Commit message: combining urdf files

File: data_processing/assets/arm/panda_delto.urdf (robot description, URDF)
Before this commit: robot panda, 11 links, 10 joints
Links:
- link panda_hand: geometry collision mesh filename=package://meshes/collision/hand.obj; visual mesh filename=package://meshes/visual/hand.obj
