Commit message: combined panda arm and gripper

File: data_processing/assets/franka_description/robots/frankaEmikaPanda.urdf (robot description, URDF)
Before this commit: robot panda, 25 links, 24 joints
Links:
- link panda_link8: mass 0.0 -> None
Joints:
- removed joint panda_hand_joint
- added joint delto_base_joint: type fixed, parent panda_link8, child delto_base_link, origin xyz=0 0 0.0502 rpy=0 0 0

Commit message: added python file testing combined urdf

File: data_processing/assets/franka_description/robots/frankaEmikaPanda.urdf (robot description, URDF)
Before this commit: robot panda, 25 links, 24 joints
Joints:
- joint delto_base_joint: origin xyz=0 0 0.0502 rpy=0 0 0 -> xyz=0 0 0.05218562175888181 rpy=0 0 0
