Commit message: Added offset to tesollo gripper urdf and xml
Added offset link to position gripper's base

File: data_processing/assets/hand/delto_gripper_3f.urdf (robot description, URDF)
Before this commit: robot delto_gripper_3f, 16 links, 15 joints
Links:
- added link offset, mass 0.0
Joints:
- added joint delto_base_joint: type fixed, parent offset, child delto_base_link, origin xyz=0 0 0.05218562175888181 rpy=0 0 0
